Commit message: fixed simulation launcher in a1_description package

File: src/a1_description/urdf/a1.urdf (robot description, URDF)
Before this commit: robot a1_description, 23 links, 22 joints
Links:
- link FL_thigh_shoulder: mass None -> 0.0
- link FR_thigh_shoulder: mass None -> 0.0
- link RL_thigh_shoulder: mass None -> 0.0
- link RR_thigh_shoulder: mass None -> 0.0
- link trunk: mass 4.713 -> 6.0
Joints:
- joint FL_calf_joint: limit lower=-2.69653369433 upper=-0.916297857297 effort=55 velocity=28.6 -> lower=-2.69653369433 upper=-0.916297857297 effort=33.5 velocity=21
- joint FL_hip_joint: limit lower=-0.802851455917 upper=0.802851455917 effort=20 velocity=52.4 -> lower=-0.802851455917 upper=0.802851455917 effort=33.5 velocity=21; origin xyz=0.183 0.047 0 rpy=0 0 0 -> xyz=0.1805 0.047 0 rpy=0 0 0
- joint FL_thigh_joint: limit lower=-1.0471975512 upper=4.18879020479 effort=55 velocity=28.6 -> lower=-1.0471975512 upper=4.18879020479 effort=33.5 velocity=21; origin xyz=0 0.08505 0 rpy=0 0 0 -> xyz=0 0.0838 0 rpy=0 0 0
- joint FR_calf_joint: limit lower=-2.69653369433 upper=-0.916297857297 effort=55 velocity=28.6 -> lower=-2.69653369433 upper=-0.916297857297 effort=33.5 velocity=21
- joint FR_hip_joint: limit lower=-0.802851455917 upper=0.802851455917 effort=20 velocity=52.4 -> lower=-0.802851455917 upper=0.802851455917 effort=33.5 velocity=21; origin xyz=0.183 -0.047 0 rpy=0 0 0 -> xyz=0.1805 -0.047 0 rpy=0 0 0
- joint FR_thigh_joint: limit lower=-1.0471975512 upper=4.18879020479 effort=55 velocity=28.6 -> lower=-1.0471975512 upper=4.18879020479 effort=33.5 velocity=21; origin xyz=0 -0.08505 0 rpy=0 0 0 -> xyz=0 -0.0838 0 rpy=0 0 0
- joint RL_calf_joint: limit lower=-2.69653369433 upper=-0.916297857297 effort=55 velocity=28.6 -> lower=-2.69653369433 upper=-0.916297857297 effort=33.5 velocity=21
- joint RL_hip_joint: limit lower=-0.802851455917 upper=0.802851455917 effort=20 velocity=52.4 -> lower=-0.802851455917 upper=0.802851455917 effort=33.5 velocity=21; origin xyz=-0.183 0.047 0 rpy=0 0 0 -> xyz=-0.1805 0.047 0 rpy=0 0 0
- joint RL_thigh_joint: limit lower=-1.0471975512 upper=4.18879020479 effort=55 velocity=28.6 -> lower=-1.0471975512 upper=4.18879020479 effort=33.5 velocity=21; origin xyz=0 0.08505 0 rpy=0 0 0 -> xyz=0 0.0838 0 rpy=0 0 0
- joint RR_calf_joint: limit lower=-2.69653369433 upper=-0.916297857297 effort=55 velocity=28.6 -> lower=-2.69653369433 upper=-0.916297857297 effort=33.5 velocity=21
- joint RR_hip_joint: limit lower=-0.802851455917 upper=0.802851455917 effort=20 velocity=52.4 -> lower=-0.802851455917 upper=0.802851455917 effort=33.5 velocity=21; origin xyz=-0.183 -0.047 0 rpy=0 0 0 -> xyz=-0.1805 -0.047 0 rpy=0 0 0
- joint RR_thigh_joint: limit lower=-1.0471975512 upper=4.18879020479 effort=55 velocity=28.6 -> lower=-1.0471975512 upper=4.18879020479 effort=33.5 velocity=21; origin xyz=0 -0.08505 0 rpy=0 0 0 -> xyz=0 -0.0838 0 rpy=0 0 0

File: src/a1_description/xacro/const.xacro (robot description, xacro)
@@ -20,72 +20,72 @@
     <xacro:property name="stick_length" value="0.2"/>
     <!-- kinematic value -->
-    <xacro:property name="thigh_offset" value="0.08505"/>
+    <xacro:property name="thigh_offset" value="0.0838"/>
     <xacro:property name="thigh_length" value="0.2"/>
     <xacro:property name="calf_length" value="0.2"/>
     <!-- leg offset from trunk center value -->
-    <xacro:property name="leg_offset_x" value="0.183"/>
+    <xacro:property name="leg_offset_x" value="0.1805"/>
     <xacro:property name="leg_offset_y" value="0.047"/>
     <xacro:property name="trunk_offset_z" value="0.01675"/>
     <xacro:property name="hip_offset" value="0.065"/>
     <!-- joint limits -->
-    <xacro:property name="damping" value="0"/>
+    <xacro:property name="damping" value="1.0"/>
     <xacro:property name="friction" value="0"/>
     <xacro:property name="hip_max" value="46"/>
     <xacro:property name="hip_min" value="-46"/>
-    <xacro:property name="hip_velocity_max" value="52.4"/>
-    <xacro:property name="hip_torque_max" value="20"/>
+    <xacro:property name="hip_velocity_max" value="21"/>
+    <xacro:property name="hip_torque_max" value="33.5"/>
     <xacro:property name="thigh_max" value="240"/>
     <xacro:property name="thigh_min" value="-60"/>
-    <xacro:property name="thigh_velocity_max" value="28.6"/>
-    <xacro:property name="thigh_torque_max" value="55"/>
+    <xacro:property name="thigh_velocity_max" value="21"/>
+    <xacro:property name="thigh_torque_max" value="33.5"/>
     <xacro:property name="calf_max" value="-52.5"/>
     <xacro:property name="calf_min" value="-154.5"/>
-    <xacro:property name="calf_velocity_max" value="28.6"/>
-    <xacro:property name="calf_torque_max" value="55"/>
-    <!-- dynamics inertial value -->
+    <xacro:property name="calf_velocity_max" value="21"/>
+    <xacro:property name="calf_torque_max" value="33.5"/>
+    <!-- dynamics inertial value        total 13.9kg -->
     <!-- trunk -->
-    <xacro:property name="trunk_mass" value="4.713"/>
-    <xacro:property name="trunk_com_x" value="0.012731"/>
-    <xacro:property name="trunk_com_y" value="0.002186"/>
-    <xacro:property name="trunk_com_z" value="0.000515"/>
-    <xacro:property name="trunk_ixx" value="0.016839930"/>
-    <xacro:property name="trunk_ixy" value="0.000083902"/>
-    <xacro:property name="trunk_ixz" value="0.000597679"/>
-    <xacro:property name="trunk_iyy" value="0.056579028"/>
-    <xacro:property name="trunk_iyz" value="0.000025134"/>
-    <xacro:property name="trunk_izz" value="0.064713601"/>
+    <xacro:property name="trunk_mass" value="6.0"/>
+    <xacro:property name="trunk_com_x" value="0.0000"/>
+    <xacro:property name="trunk_com_y" value="0.0041"/>
+    <xacro:property name="trunk_com_z" value="-0.0005"/>
+    <xacro:property name="trunk_ixx" value="0.0158533"/>
+    <xacro:property name="trunk_ixy" value="-0.0000366"/>
+    <xacro:property name="trunk_ixz" value="-0.0000611"/>
+    <xacro:property name="trunk_iyy" value="0.0377999"/>
+    <xacro:property name="trunk_iyz" value="-0.0000275"/>
+    <xacro:property name="trunk_izz" value="0.0456542"/>
     <!-- hip (left front) -->
-    <xacro:property name="hip_mass" value="0.696"/>
-    <xacro:property name="hip_com_x" value="-0.003311"/>
-    <xacro:property name="hip_com_y" value="0.000635"/>
-    <xacro:property name="hip_com_z" value="0.000031"/>
-    <xacro:property name="hip_ixx" value="0.000469246"/>
-    <xacro:property name="hip_ixy" value="-0.000009409"/>
-    <xacro:property name="hip_ixz" value="-0.000000342"/>
-    <xacro:property name="hip_iyy" value="0.000807490"/>
-    <xacro:property name="hip_iyz" value="-0.000000466"/>
-    <xacro:property name="hip_izz" value="0.000552929"/>
+    <xacro:property name="hip_mass" value="0.595"/>
+    <xacro:property name="hip_com_x" value="-0.003875"/>
+    <xacro:property name="hip_com_y" value="0.001622"/>
+    <xacro:property name="hip_com_z" value="0.000042"/>
+    <xacro:property name="hip_ixx" value="0.000402747"/>
+    <xacro:property name="hip_ixy" value="-0.000008709"/>
+    <xacro:property name="hip_ixz" value="-0.000000297"/>
+    <xacro:property name="hip_iyy" value="0.000691123"/>
+    <xacro:property name="hip_iyz" value="-0.000000545"/>
+    <xacro:property name="hip_izz" value="0.000487919"/>
     <!-- thigh -->
-    <xacro:property name="thigh_mass" value="1.013"/>
-    <xacro:property name="thigh_com_x" value="-0.003237"/>
-    <xacro:property name="thigh_com_y" value="-0.022327"/>
-    <xacro:property name="thigh_com_z" value="-0.027326"/>
-    <xacro:property name="thigh_ixx" value="0.005529065"/>
-    <xacro:property name="thigh_ixy" value="0.000004825"/>
-    <xacro:property name="thigh_ixz" value="0.000343869"/>
-    <xacro:property name="thigh_iyy" value="0.005139339"/>
-    <xacro:property name="thigh_iyz" value="0.000022448"/>
-    <xacro:property name="thigh_izz" value="0.001367788"/>
+    <xacro:property name="thigh_mass" value="0.888"/>
+    <xacro:property name="thigh_com_x" value="-0.003574"/>
+    <xacro:property name="thigh_com_y" value="-0.019529"/>
+    <xacro:property name="thigh_com_z" value="-0.030323"/>
+    <xacro:property name="thigh_ixx" value="0.005251806"/>
+    <xacro:property name="thigh_ixy" value="-0.000002168"/>
+    <xacro:property name="thigh_ixz" value="0.000346889"/>
+    <xacro:property name="thigh_iyy" value="0.005000475"/>
+    <xacro:property name="thigh_iyz" value="-0.000028174"/>
+    <xacro:property name="thigh_izz" value="0.001110200"/>
     <!-- calf -->
-    <xacro:property name="calf_mass" value="0.166"/>
-    <xacro:property name="calf_com_x" value="0.006435"/>
-    <xacro:property name="calf_com_y" value="0.0"/>
-    <xacro:property name="calf_com_z" value="-0.107388"/>
-    <xacro:property name="calf_ixx" value="0.002997972"/>
+    <xacro:property name="calf_mass" value="0.151"/>
+    <xacro:property name="calf_com_x" value="0.007105"/>
+    <xacro:property name="calf_com_y" value="-0.000239"/>
+    <xacro:property name="calf_com_z" value="-0.096933"/>
+    <xacro:property name="calf_ixx" value="0.002344758"/>
     <xacro:property name="calf_ixy" value="0.0"/>
-    <xacro:property name="calf_ixz" value="-0.000141163"/>
-    <xacro:property name="calf_iyy" value="0.003014022"/>
+    <xacro:property name="calf_ixz" value="-0.000141275"/>
+    <xacro:property name="calf_iyy" value="0.002360755"/>
     <xacro:property name="calf_iyz" value="0.0"/>
-    <xacro:property name="calf_izz" value="0.000032426"/>
+    <xacro:property name="calf_izz" value="0.000031158"/>
     <!-- foot -->
     <xacro:property name="foot_mass" value="0.06"/>

File: src/a1_description/xacro/leg.xacro (robot description, xacro)
@@ -31,5 +31,5 @@
                 </xacro:if>
                 <geometry>
-                    <mesh filename="package://a1_description/meshes/hip.dae" scale="1 1 1"/>
+                    <mesh filename="$(find a1_description)/meshes/hip.dae" scale="1 1 1"/>
                 </geometry>
                 <material name="orange"/>
@@ -77,8 +77,8 @@
                 <geometry>
                     <xacro:if value="${mirror_dae == True}">
-                        <mesh filename="package://a1_description/meshes/thigh.dae" scale="1 1 1"/>
+                        <mesh filename="$(find a1_description)/meshes/thigh.dae" scale="1 1 1"/>
                     </xacro:if>
                     <xacro:if value="${mirror_dae == False}">
-                        <mesh filename="package://a1_description/meshes/thigh_mirror.dae" scale="1 1 1"/>
+                        <mesh filename="$(find a1_description)/meshes/thigh_mirror.dae" scale="1 1 1"/>
                     </xacro:if>
                 </geometry>
@@ -112,5 +112,5 @@
                 <origin rpy="0 0 0" xyz="0 0 0"/>
                 <geometry>
-                    <mesh filename="package://a1_description/meshes/calf.dae" scale="1 1 1"/>
+                    <mesh filename="$(find a1_description)/meshes/calf.dae" scale="1 1 1"/>
                 </geometry>
                 <material name="orange"/>

File: src/a1_description/xacro/robot.xacro (robot description, xacro)
@@ -1,13 +1,16 @@
 <?xml version="1.0"?>
 <robot name="a1_description" xmlns:xacro="http://www.ros.org/wiki/xacro">
+    <xacro:arg name="use_gazebo" default="false"/>
+    <xacro:arg name="DEBUG" default="false"/>
     <xacro:include filename="$(find a1_description)/xacro/const.xacro"/>
     <xacro:include filename="$(find a1_description)/xacro/materials.xacro"/>
     <xacro:include filename="$(find a1_description)/xacro/leg.xacro"/>
     <xacro:include filename="$(find a1_description)/xacro/stairs.xacro"/>
-    <!-- <xacro:include filename="$(find a1_gazebo)/launch/gazebo.xacro"/> -->
+    <xacro:include filename="$(find a1_description)/xacro/gazebo.xacro"/>
+    <xacro:include filename="$(find a1_description)/xacro/ros2_control.xacro"/>
     <!-- <xacro:include filename="$(find a1_gazebo)/launch/stairs.urdf.xacro"/> -->
     <!-- <xacro:stairs stairs="15" xpos="0" ypos="0" zpos="0" /> -->
     <!-- Rollover Protection mode will add an additional stick on the top, use "true" or "false" to switch it. -->
-    <xacro:property name="rolloverProtection" value="false"/>
+    <xacro:property name="rolloverProtection" value="true"/>
     <!-- Debug mode will hung up the robot, use "true" or "false" to switch it. -->
     <xacro:if value="$(arg DEBUG)">
@@ -36,5 +39,5 @@
             <origin rpy="0 0 0" xyz="0 0 0"/>
             <geometry>
-                <mesh filename="package://a1_description/meshes/trunk.dae" scale="1 1 1"/>
+                <mesh filename="$(find a1_description)/meshes/trunk.dae" scale="1 1 1"/>
             </geometry>
             <material name="orange"/>
@@ -121,4 +124,88 @@
         <origin rpy="0 0 0" xyz="${-leg_offset_x} ${leg_offset_y} 0"/>
     </xacro:leg>
-    <!-- <xacro:stairs stairs="15" xpos="0" ypos="2.0" zpos="0" /> -->
+    <xacro:unless value="$(arg use_gazebo)">
+        <ros2_control name="a1_ros2_control_settings" type="system">
+            <hardware>
+                <plugin>unitree_hardware/UnitreeHardware</plugin>
+            </hardware>
+            <xacro:leg_ros2_control leg_name="FL"/>
+            <xacro:leg_ros2_control leg_name="FR"/>
+            <xacro:leg_ros2_control leg_name="RL"/>
+            <xacro:leg_ros2_control leg_name="RR"/>
+            <sensor name="imu_sensor">
+                <state_interface name="orientation.x"/>
+                <state_interface name="orientation.y"/>
+                <state_interface name="orientation.z"/>
+                <state_interface name="orientation.w"/>
+                <state_interface name="angular_velocity.x"/>
+                <state_interface name="angular_velocity.y"/>
+                <state_interface name="angular_velocity.z"/>
+                <state_interface name="linear_acceleration.x"/>
+                <state_interface name="linear_acceleration.y"/>
+                <state_interface name="linear_acceleration.z"/>
+            </sensor>
+            <sensor name="FL_foot_force_sensor">
+                <frame_id name="FL_foot"/>
+                <state_interface name="force.z"/>
+            </sensor>
+            <sensor name="FR_foot_force_sensor">
+                <frame_id name="FR_foot"/>
+                <state_interface name="force.z"/>
+            </sensor>
+            <sensor name="RL_foot_force_sensor">
+                <frame_id name="RL_foot"/>
+                <state_interface name="force.z"/>
+            </sensor>
+            <sensor name="RR_foot_force_sensor">
+                <frame_id name="RR_foot"/>
+                <state_interface name="force.z"/>
+            </sensor>
+        </ros2_control>
+    </xacro:unless>
+    <xacro:if value="$(arg use_gazebo)">
+        <ros2_control name="a1_ros2_control_settings" type="system">
+            <hardware>
+                <plugin>unitree_gazebo/UnitreeGazeboSystem</plugin>
+                <!-- <plugin>gazebo_ros2_control/GazeboSystem</plugin> since we have modified version in unitree_gazebo-->
+            </hardware>
+            <xacro:leg_ros2_control leg_name="FL"/>
+            <xacro:leg_ros2_control leg_name="FR"/>
+            <xacro:leg_ros2_control leg_name="RL"/>
+            <xacro:leg_ros2_control leg_name="RR"/>
+            <sensor name="imu_sensor">
+                <state_interface name="orientation.x"/>
+                <state_interface name="orientation.y"/>
+                <state_interface name="orientation.z"/>
+                <state_interface name="orientation.w"/>
+                <state_interface name="angular_velocity.x"/>
+                <state_interface name="angular_velocity.y"/>
+                <state_interface name="angular_velocity.z"/>
+                <state_interface name="linear_acceleration.x"/>
+                <state_interface name="linear_acceleration.y"/>
+                <state_interface name="linear_acceleration.z"/>
+            </sensor>
+            <sensor name="FL_foot_force_sensor">
+                <frame_id name="FL_foot"/>
+                <state_interface name="force.z"/>
+            </sensor>
+            <sensor name="FR_foot_force_sensor">
+                <frame_id name="FR_foot"/>
+                <state_interface name="force.z"/>
+            </sensor>
+            <sensor name="RL_foot_force_sensor">
+                <frame_id name="RL_foot"/>
+                <state_interface name="force.z"/>
+            </sensor>
+            <sensor name="RR_foot_force_sensor">
+                <frame_id name="RR_foot"/>
+                <state_interface name="force.z"/>
+            </sensor>
+        </ros2_control>
+        <gazebo>
+            <plugin filename="libgazebo_ros2_control.so" name="gazebo_ros2_control">
+                <robot_sim_type>    </robot_sim_type>
+                <!-- <parameters>$(find unitree_controller)/config/a1_gazebo_controllers.yaml</parameters> -->
+            </plugin>
+        </gazebo>
+    </xacro:if>
 </robot>
